Commit message: use world file for static scene; fix Kinect pose + spawn ordering
- worlds/ur5e_scene.world bakes in sun + ground + ur5_base + cafe_table
  via model:// URIs. Removes the launch-level spawn races for static
  models and the launch now only spawns things the RL env may need to
  reset (cube + arm).
- ur5e_robotiq85_kinect.urdf.xacro: Kinect pose now mirrors the RX200
  convention (front of workspace, looking back) offset by the
  cafe-table x=0.7 so the cube workspace is centred in frame.
- launch: add output=screen on spawn_cube so missing-file / parse
  errors surface in the terminal.
- CMakeLists install: include worlds/ alongside config/launch/models/urdf.

File: urdf/ur5e_robotiq85_kinect.urdf.xacro (robot description, xacro)
@@ -2,9 +2,9 @@
 <!--
   UR5e + Robotiq 2F-85 + head-mount Kinect v2.
-  Kinect is mounted to the URDF `world` frame so its pose is in
-  Gazebo world coordinates, not affected by the spawn offset of the
-  arm. The default <origin> below puts it ~1.6 m above the workspace,
-  tilted ~45 degrees toward the cafe-table top at (0.7, 0, 0.775).
-  Adjust to taste — RL envs subscribe to /kinect2/* regardless.
+  Kinect mounts to the URDF `world` frame (Gazebo world coordinates,
+  unaffected by the arm's spawn offset). Pose mirrors RX200's
+  rx200_kinect.urdf.xacro convention (camera in front, looking back
+  toward the workspace), offset by the cafe-table x = 0.7 so the
+  cube workspace is centred in frame.
 -->
 <robot xmlns:xacro="http://www.ros.org/wiki/xacro" name="ur5e_robotiq_85_kinect">
@@ -12,5 +12,5 @@
   <xacro:include filename="$(find common_sensors)/urdf/sensors/kinect2.urdf.xacro"/>
   <xacro:kinect2 name="kinect2" parent="world">
-    <origin rpy="0 0.8 0" xyz="1.5 0 1.5"/>
+    <origin rpy="0 0.3 3.15" xyz="2.1 -0.08 0.9"/>
   </xacro:kinect2>
 </robot>
